Commit message: update: change path for ur10e_rg2_moveit package and modify .gitignore files

File: ROS/src/ur10e_rg2_moveit/config/gazebo_ur10e_robot_rg2.urdf (robot description, URDF)
Before this commit: robot ur10e_robot_rg2, 17 links, 16 joints
Links:
- link base_link_inertia: geometry collision mesh filename=package://ur10e_rg2_urdf/meshes/ur10e/collision/base.stl; visual mesh filename=package://ur10e_rg2_urdf/meshes/ur10e/visual/base.dae
- link forearm_link: geometry collision mesh filename=package://ur10e_rg2_urdf/meshes/ur10e/collision/forearm.stl; visual mesh filename=package://ur10e_rg2_urdf/meshes/ur10e/visual/forearm.dae
- link left_inner_finger: geometry collision mesh filename=package://ur10e_rg2_urdf/meshes/rg2/collision/inner_finger.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; visual mesh filename=package://ur10e_rg2_urdf/meshes/rg2/visual/inner_finger.stl
- link left_inner_knuckle: geometry collision mesh filename=package://ur10e_rg2_urdf/meshes/rg2/collision/inner_knuckle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; visual mesh filename=package://ur10e_rg2_urdf/meshes/rg2/visual/inner_knuckle.stl
- link left_outer_knuckle: geometry collision mesh filename=package://ur10e_rg2_urdf/meshes/rg2/collision/outer_knuckle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; visual mesh filename=package://ur10e_rg2_urdf/meshes/rg2/visual/outer_knuckle.stl
- link onrobot_rg2_base_link: geometry collision mesh filename=package://ur10e_rg2_urdf/meshes/rg2/collision/base_link.stl; visual mesh filename=package://ur10e_rg2_urdf/meshes/rg2/visual/base_link.stl
- link right_inner_finger: geometry collision mesh filename=package://ur10e_rg2_urdf/meshes/rg2/collision/inner_finger.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; visual mesh filename=package://ur10e_rg2_urdf/meshes/rg2/visual/inner_finger.stl
- link right_inner_knuckle: geometry collision mesh filename=package://ur10e_rg2_urdf/meshes/rg2/collision/inner_knuckle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; visual mesh filename=package://ur10e_rg2_urdf/meshes/rg2/visual/inner_knuckle.stl
- link right_outer_knuckle: geometry collision mesh filename=package://ur10e_rg2_urdf/meshes/rg2/collision/outer_knuckle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; visual mesh filename=package://ur10e_rg2_urdf/meshes/rg2/visual/outer_knuckle.stl
- link shoulder_link: geometry collision mesh filename=package://ur10e_rg2_urdf/meshes/ur10e/collision/shoulder.stl; visual mesh filename=package://ur10e_rg2_urdf/meshes/ur10e/visual/shoulder.dae
- link upper_arm_link: geometry collision mesh filename=package://ur10e_rg2_urdf/meshes/ur10e/collision/upperarm.stl; visual mesh filename=package://ur10e_rg2_urdf/meshes/ur10e/visual/upperarm.dae
- link wrist_1_link: geometry collision mesh filename=package://ur10e_rg2_urdf/meshes/ur10e/collision/wrist1.stl; visual mesh filename=package://ur10e_rg2_urdf/meshes/ur10e/visual/wrist1.dae
- link wrist_2_link: geometry collision mesh filename=package://ur10e_rg2_urdf/meshes/ur10e/collision/wrist2.stl; visual mesh filename=package://ur10e_rg2_urdf/meshes/ur10e/visual/wrist2.dae
- link wrist_3_link: geometry collision mesh filename=package://ur10e_rg2_urdf/meshes/ur10e/collision/wrist3.stl; visual mesh filename=package://ur10e_rg2_urdf/meshes/ur10e/visual/wrist3.dae
